File: hardware/pico_dual_PMSM_BUG79100G_DRV8316C.kicad_pcb (KiCad board)
At the start: 4 copper layers, 55 x 60 mm, 85 parts, among them IC1 BU79100G-LATR, IC2 BU79100G-LATR, IC3 BU79100G-LATR, IC4 BU79100G-LATR, IC5 THVD2450DRBR, J10 BM06B-SRSS-TB, J11 BM06B-SRSS-TB, J12 DF13-02P-1.25DSA, J14 Conn_01x01_Pin, J15 Conn_01x01_Pin, J16 Conn_01x01_Pin, J17 Conn_01x01_Pin, J18 Conn_01x01_Pin, J19 Conn_01x01_Pin, J2 XT30PW-M, J20 Conn_01x01_Pin, J21 Conn_01x01_Pin, J22 Conn_01x01_Pin, J23 Conn_01x01_Pin, J24 Conn_01x01_Pin, J25 Conn_01x01_Pin, SW1 PTS810SJM250SMTRLFS, U1 DRV8316CRRGFR, U3 DRV8316CRRGFR

Commit message: Add mouser part number, height for openpnp, fix silkscreen.
Other:
- board text removed: "SCK MISO MOSI CS VCC GND"
