File: hardware/pico_dual_PMSM_BUG79100G_DRV8316C.kicad_sch (KiCad schematic)
At the start: 68 parts, among them IC1 BU79100G-LATR, IC2 BU79100G-LATR, IC3 BU79100G-LATR, IC4 BU79100G-LATR, IC5 THVD2450DRBR, J10 Conn_01x06, J11 Conn_01x06, J12 Conn_01x02_Pin, J2 Conn_01x02, U1 DRV8316CRRGFR, U3 DRV8316CRRGFR

Commit message: update pcb
Parts:
- C2, C8: value C -> 1uF 50V
- C21, C23, C24, C25, C3: value 100nF -> 100n
- C5: value C -> 100nF
- C9: value 100uF -> 100uF 50V
Changed lines of the file:
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@@
 			)
 		)
-		(property "Value" "C"
+		(property "Value" "1uF 50V"
 			(at 60.96 138.4301 0)
 			(show_name no)
@@
 			)
 		)
-		(property "Value" "100nF"
+		(property "Value" "100n"
 			(at 53.594 206.756 90)
 			(show_name no)
@@
 			)
 		)
-		(property "Value" "C"
+		(property "Value" "1uF 50V"
 			(at 76.2 138.4301 0)
 			(show_name no)
@@
 			)
 		)
-		(property "Value" "100nF"
+		(property "Value" "100n"
 			(at 151.13 86.106 90)
 			(show_name no)
@@
 			)
 		)
-		(property "Value" "C"
+		(property "Value" "100nF"
 			(at 266.7 198.12 0)
 			(show_name no)
@@
 			)
 		)
-		(property "Value" "100nF"
+		(property "Value" "100n"
 			(at 225.044 52.07 90)
 			(show_name no)
@@
 			)
 		)
-		(property "Value" "100nF"
+		(property "Value" "100n"
 			(at 223.774 124.46 90)
 			(show_name no)
@@
 			)
 		)
-		(property "Value" "100uF"
+		(property "Value" "100uF 50V"
 			(at 86.36 140.0809 0)
 			(show_name no)
@@
 			)
 		)
-		(property "Value" "100nF"
+		(property "Value" "100n"
 			(at 53.594 180.086 90)
 			(show_name no)

Commit message: add board diag at boot (press '?' at boot to test)
Parts:
- added C10: 1uF 50V, Capacitor_SMD:C_1206_3216Metric, symbol Device:C
- added C26: 100n, Capacitor_SMD:C_0402_1005Metric, symbol Device:C
- added D1: SK6812MINI, LED_SMD:LED_SK6812MINI_PLCC4_3.5x3.5mm_P1.75mm, symbol LED:SK6812MINI
- added J14, J15, J16, J17, J18, J19, J20, J21, J22, J23, J24, J25: Conn_01x01_Pin, Connector_Wire:SolderWirePad_1x01_SMD_1x2mm, symbol Connector:Conn_01x01_Pin
- added R29: 330, Resistor_SMD:R_0402_1005Metric, symbol Device:R
- added SW1: PTS810SJM250SMTRLFS, Button_Switch_SMD:SW_SPST_PTS810, symbol Switch:SW_Push
- A1, J4, J5, J6, J7, J8, J9: now left out of the parts list
- C15, C16, C17, C18: value 22p -> 100p
- C2, C8: footprint Capacitor_SMD:C_1812_4532Metric -> Capacitor_SMD:C_1206_3216Metric
- J10, J11: value Conn_01x06 -> BM06B-SRSS-TB
- J12: value Conn_01x02_Pin -> DF13-02P-1.25DSA
- J2: value Conn_01x02 -> XT30PW-M
Connections:
- net GND: now also J10.6 (Pin_6), J11.6 (Pin_6), C10.1, C26.1, D1.2 (VSS), J20.1 (Pin_1), J25.1 (Pin_1), SW1.1; no longer J10.1 (Pin_1), J11.1 (Pin_1)
- net M0_ENC_CLK: now also J10.1 (Pin_1), J14.1 (Pin_1); no longer J10.5 (Pin_5)
- net M0_ENC_CS: now also J10.4 (Pin_4), J17.1 (Pin_1); no longer J10.6 (Pin_6)
- net M0_ENC_MISO: now also J10.2 (Pin_2), J11.2 (Pin_2), J15.1 (Pin_1), J21.1 (Pin_1); no longer J10.3 (Pin_3), J11.3 (Pin_3)
- net M0_ENC_MOSI: now also J10.3 (Pin_3), J16.1 (Pin_1); no longer J10.4 (Pin_4)
- net M1_ENC_CLK: now also J11.1 (Pin_1), J18.1 (Pin_1); no longer J11.5 (Pin_5)
- net M1_ENC_CS: now also J11.4 (Pin_4), J23.1 (Pin_1); no longer J11.6 (Pin_6)
- net M1_ENC_MOSI: now also J11.3 (Pin_3), J22.1 (Pin_1); no longer J11.4 (Pin_4)
- net VBUS: now also C10.2
- net VCC: now also J10.5 (Pin_5), J11.5 (Pin_5), C26.2, D1.4 (VDD), J19.1 (Pin_1), J24.1 (Pin_1); no longer J10.2 (Pin_2), J11.2 (Pin_2)
- net LED_SW: now reaches A1.34 (GPIO28_ADC2)
- net LED_SW: now also D1.3 (DIN), R29.1
- new net: R29.2, SW1.2
Other:
- note added: "4.8Mhz"
- moved on the sheet: C9

Commit message: Add mouser part number, height for openpnp, fix silkscreen.
Parts:
- A1: MPN (none) -> SC1631; Manufacturer_Name (none) -> Raspberry Pi; Manufacturer_Part_Number (none) -> SC1631; Mouser Part Number (none) -> 358-SC1631; mouser (none) -> 358-SC1631; now in the parts list
- C1, C12, C13, C21, C23, C24, C25, C26, C3, C4: Height (none) -> 0.5; MPN (none) -> CL05B104KB5NNWC; Manufacturer_Name (none) -> Samsung Electro-Mechanics; Manufacturer_Part_Number (none) -> CL05B104KB5NNWC; Mouser Part Number (none) -> 187-CL05B104KB5NNWC; mouser (none) -> 187-CL05B104KB5NNWC
- C10, C2, C8: Height (none) -> 1.8; MPN (none) -> C1206F105M5RACAUTO; Manufacturer_Name (none) -> KEMET; Manufacturer_Part_Number (none) -> C1206F105M5RACAUTO; Mouser Part Number (none) -> 80-C1206F105M5RAUTO; mouser (none) -> 80-C1206F105M5RAUTO
- C11, C20, C6, C7: Height (none) -> 0.5; MPN (none) -> CL05A105KO5NNNC; Manufacturer_Name (none) -> Samsung Electro-Mechanics; Manufacturer_Part_Number (none) -> CL05A105KO5NNNC; Mouser Part Number (none) -> 187-CL05A105KO5NNNC; mouser (none) -> 187-CL05A105KO5NNNC
- C14, C22: Height (none) -> 1.4; MPN (none) -> C0805C226M8PACTU; Manufacturer_Name (none) -> KEMET; Manufacturer_Part_Number (none) -> C0805C226M8PACTU; Mouser Part Number (none) -> 80-C0805C226M8P; mouser (none) -> 80-C0805C226M8P
- C15, C16, C17, C18: Height (none) -> 0.5; MPN C0402C104M4RAC7411 -> GRM1555C1H101JA01J; Manufacturer_Name (none) -> Murata Electronics; Manufacturer_Part_Number (none) -> GRM1555C1H101JA01J; Mouser Part Number (none) -> 81-GRM1555C1H101JA1J; mouser 80-C0402C104M4RACLR -> 81-GRM1555C1H101JA1J
- C5: Height (none) -> 0.8; MPN (none) -> GRM188R72A104KA35D; Manufacturer_Name (none) -> Murata Electronics; Manufacturer_Part_Number (none) -> GRM188R72A104KA35D; Mouser Part Number (none) -> 81-GRM188R72A104KA35; mouser (none) -> 81-GRM188R72A104KA35
- C9: MPN (none) -> MAL219051101E3; Manufacturer_Name (none) -> Vishay / BC Components; Manufacturer_Part_Number (none) -> MAL219051101E3; Mouser Part Number (none) -> 594-MAL219051101E3; mouser (none) -> 594-MAL219051101E3
- D1: Height (none) -> 0.95
- IC1, IC2, IC3, IC4: MPN (none) -> BU79100G-LATR; mouser (none) -> 755-BU79100G-LATR
- IC5: MPN (none) -> THVD2450DRBR; mouser (none) -> 595-THVD2450DRBR
- J10, J11: Height (none) -> 4.25; MPN (none) -> BM06B-SRSS-TB(LF)(SN); Manufacturer_Name (none) -> JST; Manufacturer_Part_Number (none) -> BM06B-SRSS-TB(LF)(SN); Mouser Part Number (none) -> 306-6BSRSSTBLPP; mouser (none) -> 306-6BSRSSTBLPP
- R1: Height (none) -> 0.45; MPN (none) -> RC0603FR-07120RL; Manufacturer_Name (none) -> YAGEO; Manufacturer_Part_Number (none) -> RC0603FR-07120RL; Mouser Part Number (none) -> 603-RC0603FR-07120RL; mouser (none) -> 603-RC0603FR-07120RL
- R10, R11, R12, R13, R29: Height (none) -> 0.35; MPN (none) -> RC0402FR-07330RL; Manufacturer_Name (none) -> YAGEO; Manufacturer_Part_Number (none) -> RC0402FR-07330RL; Mouser Part Number (none) -> 603-RC0402FR-07330RL; mouser (none) -> 603-RC0402FR-07330RL
- R14, R16, R23, R28: Height (none) -> 0.35; MPN (none) -> RC0402FR-0710KL; Manufacturer_Name (none) -> YAGEO; Manufacturer_Part_Number (none) -> RC0402FR-0710KL; Mouser Part Number (none) -> 603-RC0402FR-0710KL; mouser (none) -> 603-RC0402FR-0710KL
- R15, R17, R18, R19, R20, R21, R24, R25, R26, R27: Height (none) -> 0.35; MPN (none) -> RC0402FR-0722RL; Manufacturer_Name (none) -> YAGEO; Manufacturer_Part_Number (none) -> RC0402FR-0722RL; Mouser Part Number (none) -> 603-RC0402FR-0722RL; mouser (none) -> 603-RC0402FR-0722RL
- R22: Height (none) -> 0.35; MPN (none) -> RC0402FR-07100KL; Manufacturer_Name (none) -> YAGEO; Manufacturer_Part_Number (none) -> RC0402FR-07100KL; Mouser Part Number (none) -> 603-RC0402FR-07100KL; mouser (none) -> 603-RC0402FR-07100KL
- SW1: Height (none) -> 2.5; MPN (none) -> PTS810SJM250SMTR LFS; Manufacturer_Name (none) -> C&K / Littelfuse; Manufacturer_Part_Number (none) -> PTS810SJM250SMTR LFS; Mouser Part Number (none) -> 611-PTS810SJM250SMTR; mouser (none) -> 611-PTS810SJM250SMTR
- U1, U3: Height (none) -> 1; MPN (none) -> DRV8316CRRGFR; Manufacturer_Name (none) -> Texas Instruments; Manufacturer_Part_Number (none) -> DRV8316CRRGFR; Mouser Part Number (none) -> 595-DRV8316CRRGFR; mouser (none) -> 595-DRV8316CRRGFR
